Commit message: Add inertial properties to robot links in URDF

File: description/robot_core.xacro (robot description, xacro)
@@ -1,4 +1,5 @@
 <?xml version="1.0"?>
 <robot xmlns:xacro="http://www.ros.org/wiki/xacro">
+    <xacro:include filename="$(find my_bot)/description/inertial_macros.xacro"/>
     <material name="white">
         <color rgba="1 1 1 1"/>
@@ -36,4 +37,7 @@
             </geometry>
         </collision>
+        <xacro:inertial_box mass="1" x="0.3" y="0.3" z="0.15">
+            <origin xyz="0.15 0 0.075"/>
+        </xacro:inertial_box>
     </link>
     <!--LEFT WHEEL  -->
@@ -58,4 +62,7 @@
             </geometry>
         </collision>
+        <xacro:inertial_cylinder mass="0.1" length="0.04" radius="0.05">
+            <origin xyz="0 0 0"/>
+        </xacro:inertial_cylinder>
     </link>
     <!--RIGHT WHEEL  -->
@@ -80,4 +87,7 @@
             </geometry>
         </collision>
+        <xacro:inertial_cylinder mass="0.1" length="0.04" radius="0.05">
+            <origin xyz="0 0 0"/>
+        </xacro:inertial_cylinder>
     </link>
     <!-- CASTOR WHEEL  -->
@@ -101,4 +111,7 @@
             </geometry>
         </collision>
+        <xacro:inertial_sphere mass="0.1" radius="0.05">
+            <origin xyz="0 0 0"/>
+        </xacro:inertial_sphere>
     </link>
 </robot>
